Commit message: Relocate all the file and add sensor
To fit the last commmit that change the way I use dockerfile from
"copy all the folder into container" to "mount this folder", I
move all the package folders into `src/`.

Create the new package "my_sensor" which will publish reality data.
The first sensor I use is zed camera, it can send position and
orientation back, that sound amazing for me to implement slam in
real world.

In the `camera_node.py` file, I receive position data by tcp/ip
because zed sdk depends on cuda which rasberry pi 4 doesn't has. So
camera will work on other cuda supported device such as laptop.

I try to simulate lidar slam by gazebo but I forgot to add install
command into dockerfile.

File: src/my_bot/description/robot_core.xacro (robot description, xacro)
@@ -20,4 +20,12 @@
     <!-- BASE LINK -->
     <link name="base_link">
+    </link>
+    <!-- BASE_FOOTPRINT LINK -->
+    <joint name="base_footprint_joint" type="fixed">
+	<parent link="base_link"/>
+	<child link="base_footprint"/>
+	<origin xyz="0 0 0" rpy="0 0 0"/>
+    </joint>
+    <link name="base_footprint">
     </link>
     <!-- CHASSIS LINK -->

Commit message: Add exec and launch file

File: src/my_bot/description/robot_core.xacro (robot description, xacro)
@@ -57,5 +57,5 @@
     </gazebo>
     <!-- LEFT WHEEL LINK -->
-    <joint name="left_wheel_joint" type="continuous">
+    <joint name="left_wheel_joint" type="fixed">
         <parent link="base_link"/>
         <child link="left_wheel"/>
@@ -83,5 +83,5 @@
     </gazebo>
     <!-- RIGHT WHEEL LINK -->
-    <joint name="right_wheel_joint" type="continuous">
+    <joint name="right_wheel_joint" type="fixed">
         <parent link="base_link"/>
         <child link="right_wheel"/>
