Commit message: Update camera node

File: src/my_bot/description/lidar.xacro (robot description, xacro)
@@ -3,8 +3,8 @@
     <joint name="laser_joint" type="fixed">
         <parent link="chassis"/>
-        <child link="laser_frame"/>
+        <child link="laser"/>
         <origin xyz="0.1 0 0.175" rpy="0 0 0"/>
     </joint>
-    <link name="laser_frame">
+    <link name="laser">
         <visual>
             <geometry>
@@ -22,5 +22,5 @@
         </xacro:inertial_cylinder>
     </link>
-    <gazebo reference="laser_frame">
+    <gazebo reference="laser">
         <material>Gazebo/Red</material>
         <sensor name="laser" type="ray">
@@ -46,5 +46,5 @@
                 </ros>
                 <output_type>sensor_msgs/LaserScan</output_type>
-                <frame_name>laser_frame</frame_name>
+                <frame_name>laser</frame_name>
             </plugin>
         </sensor>

File: src/my_bot/description/robot_core.xacro (robot description, xacro)
@@ -57,5 +57,5 @@
     </gazebo>
     <!-- LEFT WHEEL LINK -->
-    <joint name="left_wheel_joint" type="fixed">
+    <joint name="left_wheel_joint" type="continuous">
         <parent link="base_link"/>
         <child link="left_wheel"/>
@@ -83,5 +83,5 @@
     </gazebo>
     <!-- RIGHT WHEEL LINK -->
-    <joint name="right_wheel_joint" type="fixed">
+    <joint name="right_wheel_joint" type="continuous">
         <parent link="base_link"/>
         <child link="right_wheel"/>
